File: LM35_LM317_POTE.sch (KiCad schematic (older format))
At the start: 41 parts, among them P3 CONN_02X02, P4 CONN_01X02, Q2 2N7002, Q3 2N7002, Q4 2N7002, Q5 2N7002, SW1 TEC_1, SW2 TEC_1, SW3 TEC_1, SW4 TEC_1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

Commit message: Arreglo Max3232_ok, Fuente_ok, Buttons&Leds, OK.Fuente correinte OK, Potenciometros OK y LM35 OK.
Parts:
- removed C4, C5, C6, C7: 100nF, c_0805, symbol C
- removed D6, D7, D8, D9: LED, LED-0805, symbol LED
- removed P3: CONN_02X02, symbol CONN_02X02
- removed Q2, Q3, Q4, Q5: 2N7002, SOT23GDS, symbol MOSFET_N
- removed R10, R11, R12, R14, R17, R20, R23, R9: 10k, SM0805, symbol R
- removed R13, R16, R19, R22: 330k, SM0805, symbol R
- removed R15, R18, R21, R24: 680, SM0805, symbol R
- removed R6, R7, R8: 1k, SM0805, symbol R
- removed SW1, SW2, SW3, SW4: TEC_1, PUSH_SWITCH_THT, symbol SW_PUSH
- removed U3: LM317_SOT223, symbol LM317_SOT223
- added J10, J6, J7, J8, J9: TB_1X2, symbol TB_1X2
- added P10, P6, P7, P9: CONN_01X02, symbol CONN_01X02
- added P5: CONN_02X02, symbol CONN_02X02
- added RV2, RV3, RV4, RV5: POT, symbol POT
- added U4, U5: LM317_SOT223, symbol LM317_SOT223
- added U6: LM35-LP, symbol LM35-LP
- R5: value 1k -> R; footprint SM0805 -> (none); Descripción RES 1K OHM 1/8W 5% 0805 SMD -> (none); Digikey 311-1.0KARCT-ND -> (none); Fabricante Yageo -> (none); Footprint 0805 -> (none); Nro de parte RC0805JR-071KL -> (none); Path datasheet ..PCB/EDU-NXP/Datasheets -> (none)
- renumbered P4 to P8, R25 to R6
Connections:
- net labels removed: +3,3V, LED1, LED2, LED3, LED4, PULS1, PULS2, PULS3, PULS4
- wire segments 75 -> 71
Other:
- moved on the sheet: P8, R6
