File: ciaa-nxp.sch (KiCad schematic (older format))
At the start: 14 parts

Commit message: Max3232 -ok, Fuente ok, Buttons y Leds, OK. Fuente correinte OK, Falta Potenciometros y LM35.
Parts:
- removed F1, F2, F3, F4, F5, F6: fiducial, symbol CONN_1
- removed H1, H2, H3, H4, H5, H6, H7: 4mm, symbol CONN_1
- removed J?: TB_1X2, ~, symbol TB_1X2
Connections:
- wire segments 0 -> 2
- no-connect marks 13 -> 0
Other:
- note removed: "Los GS son puentes soldables en el PCB."
- note removed: "fiduciales\n\nTOP BOTTOM"
Changed lines of the file:
@@
 $Descr A4 11693 8268
 encoding utf-8
-Sheet 1 4
+Sheet 1 6
 Title "CIAA NXP"
 Date "11 may 2015"
@@
 $EndDescr
 $Sheet
-S 4200 6150 1150 1200
+S 5550 2250 1150 1200
 U 52C1F703
 F0 "RS232_TTL" 50
 F1 "RS232_TTL.sch" 50
-F2 "TTL_RS232_TXD1" I L 4200 6300 60
-F3 "TTL_RS232_TXD2" I L 4200 6800 60
-F4 "RS232_TXD1" I R 5350 6400 60
-F5 "RS232_RXD1" O R 5350 6650 60
-F6 "TTL_RS232_RXD1" I L 4200 6550 60
-F7 "TTL_RS232_RXD2" I L 4200 7050 60
-F8 "RS232_TXD2" O R 5350 6900 60
-F9 "RS232_RXD2" I R 5350 7150 60
+F2 "TTL_RS232_TXD1" I L 5550 2400 60
+F6 "TTL_RS232_RXD1" I L 5550 2550 60
 $EndSheet
-Text Notes 8700 5350 0    60   ~ 0
-Los GS son puentes soldables en el PCB.
 Text Notes 8550 2000 0    118  ~ 0
 Índice:\n1. Esquemático jerárquico\n4. RS232\n6. GPIO\n7. Entradas digitales\n8. Salidas digitales\n9. Entradas analógicas\n12. Fuente de alimentación
-$Comp
-L CONN_1 H1
-U 1 1 533F364A
-P 8950 4300
-F 0 "H1" H 9030 4300 40  0000 L CNN
-F 1 "4mm" H 8950 4355 157 0001 C CNN
-F 2 "" H 8950 4300 60  0000 C CNN
-F 3 "" H 8950 4300 60  0000 C CNN
-	1    8950 4300
-	1    0    0    -1
-$EndComp
-$Comp
-L CONN_1 H2
-U 1 1 533F6096
-P 8950 4450
-F 0 "H2" H 9030 4450 40  0000 L CNN
-F 1 "4mm" H 8950 4505 157 0001 C CNN
-F 2 "" H 8950 4450 60  0000 C CNN
-F 3 "" H 8950 4450 60  0000 C CNN
-	1    8950 4450
-	1    0    0    -1
-$EndComp
-$Comp
-L CONN_1 H3
-U 1 1 533F609C
-P 8950 4600
-F 0 "H3" H 9030 4600 40  0000 L CNN
-F 1 "4mm" H 8950 4655 157 0001 C CNN
-F 2 "" H 8950 4600 60  0000 C CNN
-F 3 "" H 8950 4600 60  0000 C CNN
-	1    8950 4600
-	1    0    0    -1
-$EndComp
-$Comp
-L CONN_1 H4
-U 1 1 533F60A2
-P 8950 4750
-F 0 "H4" H 9030 4750 40  0000 L CNN
-F 1 "4mm" H 8950 4805 157 0001 C CNN
-F 2 "" H 8950 4750 60  0000 C CNN
-F 3 "" H 8950 4750 60  0000 C CNN
-	1    8950 4750
-	1    0    0    -1
-$EndComp
-$Comp
-L CONN_1 F1
-U 1 1 5345C5B3
-P 10000 4950
-F 0 "F1" H 10080 4950 40  0000 L CNN
-F 1 "fiducial" H 10000 5005 157 0001 C CNN
-F 2 "" H 10000 4950 60  0000 C CNN
-F 3 "" H 10000 4950 60  0000 C CNN
-	1    10000 4950
-	1    0    0    -1
-$EndComp
-$Comp
-L CONN_1 F2
-U 1 1 5345D4AD
-P 10000 5050
-F 0 "F2" H 10080 5050 40  0000 L CNN
-F 1 "fiducial" H 10000 5105 157 0001 C CNN
-F 2 "" H 10000 5050 60  0000 C CNN
-F 3 "" H 10000 5050 60  0000 C CNN
-	1    10000 5050
-	1    0    0    -1
-$EndComp
-$Comp
-L CONN_1 F3
-U 1 1 5345D4B3
-P 10000 5150
-F 0 "F3" H 10080 5150 40  0000 L CNN
-F 1 "fiducial" H 10000 5205 157 0001 C CNN
-F 2 "" H 10000 5150 60  0000 C CNN
-F 3 "" H 10000 5150 60  0000 C CNN
-	1    10000 5150
-	1    0    0    -1
-$EndComp
-$Comp
-L CONN_1 F4
-U 1 1 5345BF4A
-P 10550 4950
-F 0 "F4" H 10630 4950 40  0000 L CNN
-F 1 "fiducial" H 10550 5005 157 0001 C CNN
-F 2 "" H 10550 4950 60  0000 C CNN
-F 3 "" H 10550 4950 60  0000 C CNN
-	1    10550 4950
-	1    0    0    -1
-$EndComp
-$Comp
-L CONN_1 F5
-U 1 1 5345BF50
-P 10550 5050
-F 0 "F5" H 10630 5050 40  0000 L CNN
-F 1 "fiducial" H 10550 5105 157 0001 C CNN
-F 2 "" H 10550 5050 60  0000 C CNN
-F 3 "" H 10550 5050 60  0000 C CNN
-	1    10550 5050
-	1    0    0    -1
-$EndComp
-$Comp
-L CONN_1 F6
-U 1 1 5345BF56
-P 10550 5150
-F 0 "F6" H 10630 5150 40  0000 L CNN
-F 1 "fiducial" H 10550 5205 157 0001 C CNN
-F 2 "" H 10550 5150 60  0000 C CNN
-F 3 "" H 10550 5150 60  0000 C CNN
-	1    10550 5150
-	1    0    0    -1
-$EndComp
-Text Notes 9850 4650 0    60   ~ 0
-fiduciales\n\nTOP       BOTTOM
-$Comp
-L CONN_1 H5
-U 1 1 534892C5
-P 8950 4950
-F 0 "H5" H 9030 4950 40  0000 L CNN
-F 1 "4mm" H 8950 5005 157 0001 C CNN
-F 2 "" H 8950 4950 60  0000 C CNN
-F 3 "" H 8950 4950 60  0000 C CNN
-	1    8950 4950
-	1    0    0    -1
-$EndComp
-$Comp
-L CONN_1 H6
-U 1 1 534892CB
-P 8950 5050
-F 0 "H6" H 9030 5050 40  0000 L CNN
-F 1 "4mm" H 8950 5105 157 0001 C CNN
-F 2 "" H 8950 5050 60  0000 C CNN
-F 3 "" H 8950 5050 60  0000 C CNN
-	1    8950 5050
-	1    0    0    -1
-$EndComp
-$Comp
-L CONN_1 H7
-U 1 1 534892D1
-P 8950 5150
-F 0 "H7" H 9030 5150 40  0000 L CNN
-F 1 "4mm" H 8950 5205 157 0001 C CNN
-F 2 "" H 8950 5150 60  0000 C CNN
-F 3 "" H 8950 5150 60  0000 C CNN
-	1    8950 5150
-	1    0    0    -1
-$EndComp
-NoConn ~ 9850 4950
-NoConn ~ 9850 5050
-NoConn ~ 9850 5150
-NoConn ~ 10400 4950
-NoConn ~ 10400 5050
-NoConn ~ 10400 5150
-NoConn ~ 8800 4300
-NoConn ~ 8800 4450
-NoConn ~ 8800 4600
-NoConn ~ 8800 4750
-NoConn ~ 8800 4950
-NoConn ~ 8800 5150
-NoConn ~ 8800 5050
-$Comp
-L TB_1X2 J?
-U 1 1 581891E5
-P 700 2550
-F 0 "J?" H 650 2800 60  0000 C CNN
-F 1 "TB_1X2" H 750 2300 60  0000 C CNN
-F 2 "~" H 650 2600 60  0000 C CNN
-F 3 "~" H 650 2600 60  0000 C CNN
-	1    700  2550
-	1    0    0    -1
-$EndComp
 $Sheet
-S 2500 6250 1100 1000
+S 3900 4050 1100 1000
 U 52C2B8A1
 F0 "Fuente" 50
 F1 "fuente.sch" 50
-F3 "USB_VBUS3" I R 3600 6600 60
 $EndSheet
 $Sheet
-S 2450 4350 1100 1000
+S 3850 2150 1100 1000
 U 5819E388
 F0 "SIM800L" 50
 F1 "SIM800L.sch" 50
-F3 "USB_VBUS3" I R 3550 4700 60
+F2 "Rx_sim800" I R 4950 2400 60
+F3 "Tx_sim800" O R 4950 2550 60
+$EndSheet
+$Sheet
+S 5600 4050 1100 1000
+U 581A00B9
+F0 "LM35_LM317_POTE" 50
+F1 "LM35_LM317_POTE.sch" 50
+$EndSheet
+Wire Wire Line
+	4950 2400 5550 2400
+Wire Wire Line
+	4950 2550 5550 2550
+$Sheet
+S 8150 3550 1100 1000
+U 5819F5A0
+F0 "Buttons_Leds" 50
+F1 "Buttons_Leds.sch" 50
 $EndSheet
 $EndSCHEMATC

Commit message: Arreglo Max3232_ok, Fuente_ok, Buttons&Leds, OK.Fuente correinte OK, Potenciometros OK y LM35 OK.
Changed lines of the file:
@@
 EESchema Schematic File Version 2
-LIBS:ciaa-nxp-rescue
-LIBS:power
-LIBS:device
-LIBS:transistors
-LIBS:conn
-LIBS:linear
-LIBS:regul
-LIBS:74xx
-LIBS:cmos4000
-LIBS:adc-dac
-LIBS:memory
-LIBS:xilinx
-LIBS:microcontrollers
-LIBS:dsp
-LIBS:microchip
-LIBS:analog_switches
-LIBS:motorola
-LIBS:texas
-LIBS:intel
-LIBS:audio
-LIBS:interface
-LIBS:digital-audio
-LIBS:philips
-LIBS:display
-LIBS:cypress
-LIBS:siliconi
-LIBS:opto
-LIBS:atmel
-LIBS:contrib
-LIBS:valves
+LIBS:sensors
 LIBS:74LVC1G04GW
+LIBS:93CXX
+LIBS:BLM15HG6015N1D
+LIBS:FT2232H
+LIBS:IS42S16400F
+LIBS:LPC4337JBD144
+LIBS:MIC2025
+LIBS:PBSS5240
+LIBS:PRTR5V0U2X
+LIBS:PS2805
+LIBS:SCHA5B0200
+LIBS:Si50x
+LIBS:TJA1040
+LIBS:TXB0108
+LIBS:Transil_diode
 LIBS:amesser-ad
 LIBS:amesser-cmos4000
@@
 LIBS:audio-vlsi
 LIBS:bat54_c
-LIBS:BLM15HG6015N1D
+LIBS:capteurs
+LIBS:fqt13n06l
 LIBS:g5v2
 LIBS:lm2596
+LIBS:mcp1415
+LIBS:mcp1416
 LIBS:mcu-nxp
 LIBS:mcu-st
-LIBS:MIC2025
+LIBS:my_lab
 LIBS:net-phy
 LIBS:nsi50010yt1g
-LIBS:PRTR5V0U2X
+LIBS:pbss5240xf
 LIBS:regulators
 LIBS:rs485_rs232_can
 LIBS:s25fl032p0xmfi013
-LIBS:SCHA5B0200
-LIBS:Si50x
-LIBS:Transil_diode
+LIBS:sw_push
+LIBS:tvs
 LIBS:w_device
-LIBS:LPC4337JBD144
-LIBS:IS42S16400F
-LIBS:TXB0108
-LIBS:FT2232H
-LIBS:93CXX
-LIBS:TJA1040
-LIBS:tvs
-LIBS:PBSS5240
-LIBS:pbss5240xf
-LIBS:sw_push
-LIBS:mcp1416
-LIBS:fqt13n06l
+LIBS:74xgxx
+LIBS:74xx
+LIBS:Altera
+LIBS:ESD_Protection
+LIBS:Lattice
+LIBS:Oscillators
+LIBS:Power_Management
+LIBS:Worldsemi
+LIBS:Xicor
+LIBS:Zilog
+LIBS:ac-dc
+LIBS:actel
+LIBS:adc-dac
+LIBS:analog_devices
+LIBS:analog_switches
+LIBS:atmel
+LIBS:audio
+LIBS:brooktre
+LIBS:cmos4000
+LIBS:cmos_ieee
+LIBS:conn
+LIBS:contrib
+LIBS:cypress
+LIBS:dc-dc
+LIBS:device
+LIBS:digital-audio
+LIBS:diode
+LIBS:display
+LIBS:dsp
+LIBS:elec-unifil
+LIBS:ftdi
+LIBS:gennum
+LIBS:graphic
+LIBS:hc11
+LIBS:intel
+LIBS:interface
+LIBS:ir
+LIBS:linear
+LIBS:logo
+LIBS:maxim
+LIBS:memory
+LIBS:microchip
+LIBS:microchip_dspic33dsc
+LIBS:microchip_pic10mcu
+LIBS:microchip_pic12mcu
+LIBS:microchip_pic16mcu
+LIBS:microchip_pic18mcu
+LIBS:microchip_pic32mcu
+LIBS:microcontrollers
+LIBS:motor_drivers
+LIBS:motorola
+LIBS:msp430
+LIBS:nordicsemi
+LIBS:nxp_armmcu
+LIBS:onsemi
+LIBS:opto
+LIBS:philips
+LIBS:power
+LIBS:powerint
+LIBS:pspice
+LIBS:references
+LIBS:regul
+LIBS:relays
+LIBS:rfcom
+LIBS:silabs
+LIBS:siliconi
+LIBS:stm8
+LIBS:stm32
+LIBS:supertex
+LIBS:switches
+LIBS:texas
+LIBS:transf
+LIBS:transistors
+LIBS:ttl_ieee
+LIBS:valves
+LIBS:video
+LIBS:xilinx
 LIBS:ciaa-nxp-cache
 EELAYER 25 0
@@
 F1 "RS232_TTL.sch" 50
 F2 "TTL_RS232_TXD1" I L 5550 2400 60
-F6 "TTL_RS232_RXD1" I L 5550 2550 60
+F3 "TTL_RS232_RXD1" I L 5550 2550 60
 $EndSheet
 Text Notes 8550 2000 0    118  ~ 0
@@
 	4950 2550 5550 2550
 $Sheet
-S 8150 3550 1100 1000
+S 7500 3250 1100 1000
 U 5819F5A0
 F0 "Buttons_Leds" 50
