File: fuente.sch (KiCad schematic (older format))
At the start: 17 parts

Commit message: Max3232 -ok, Fuente ok, Buttons y Leds, OK. Fuente correinte OK, Falta Potenciometros y LM35.
Parts:
- added P6: USB_OTG, symbol USB_OTG
- gave numbers to parts that had none: 17
Connections:
- net labels removed: USB_VBUS3
- wire segments 45 -> 47
- no-connect marks 0 -> 4
Other:
- moved on the sheet: U2

Commit message: Arreglo Max3232_ok, Fuente_ok, Buttons&Leds, OK.Fuente correinte OK, Potenciometros OK y LM35 OK.
Parts:
- P2: renamed from P6; symbol USB_OTG -> USB_OTG-RESCUE-ciaa-nxp
- TH1: symbol THERMISTOR -> THERMISTOR-RESCUE-ciaa-nxp
- U3: renamed from U2; symbol NCP1117ST33T3G -> NCP1117ST33T3G-RESCUE-ciaa-nxp
- renumbered C1 to C6, C2 to C7, C3 to C8, J2 to J5, U1 to U2
Changed lines of the file:
@@
 EESchema Schematic File Version 2
-LIBS:ciaa-nxp-rescue
-LIBS:power
-LIBS:device
-LIBS:transistors
-LIBS:conn
-LIBS:linear
-LIBS:regul
-LIBS:74xx
-LIBS:cmos4000
-LIBS:adc-dac
-LIBS:memory
-LIBS:xilinx
-LIBS:microcontrollers
-LIBS:dsp
-LIBS:microchip
-LIBS:analog_switches
-LIBS:motorola
-LIBS:texas
-LIBS:intel
-LIBS:audio
-LIBS:interface
-LIBS:digital-audio
-LIBS:philips
-LIBS:display
-LIBS:cypress
-LIBS:siliconi
-LIBS:opto
-LIBS:atmel
-LIBS:contrib
-LIBS:valves
+LIBS:sensors
 LIBS:74LVC1G04GW
+LIBS:93CXX
+LIBS:BLM15HG6015N1D
+LIBS:FT2232H
+LIBS:IS42S16400F
+LIBS:LPC4337JBD144
+LIBS:MIC2025
+LIBS:PBSS5240
+LIBS:PRTR5V0U2X
+LIBS:PS2805
+LIBS:SCHA5B0200
+LIBS:Si50x
+LIBS:TJA1040
+LIBS:TXB0108
+LIBS:Transil_diode
 LIBS:amesser-ad
 LIBS:amesser-cmos4000
@@
 LIBS:audio-vlsi
 LIBS:bat54_c
-LIBS:BLM15HG6015N1D
+LIBS:capteurs
+LIBS:fqt13n06l
 LIBS:g5v2
 LIBS:lm2596
+LIBS:mcp1415
+LIBS:mcp1416
 LIBS:mcu-nxp
 LIBS:mcu-st
-LIBS:MIC2025
+LIBS:my_lab
 LIBS:net-phy
 LIBS:nsi50010yt1g
-LIBS:PRTR5V0U2X
+LIBS:pbss5240xf
 LIBS:regulators
 LIBS:rs485_rs232_can
 LIBS:s25fl032p0xmfi013
-LIBS:SCHA5B0200
-LIBS:Si50x
-LIBS:Transil_diode
+LIBS:sw_push
+LIBS:tvs
 LIBS:w_device
-LIBS:LPC4337JBD144
-LIBS:IS42S16400F
-LIBS:TXB0108
-LIBS:FT2232H
-LIBS:93CXX
-LIBS:TJA1040
-LIBS:tvs
-LIBS:PBSS5240
-LIBS:pbss5240xf
-LIBS:sw_push
-LIBS:mcp1416
-LIBS:fqt13n06l
+LIBS:74xgxx
+LIBS:74xx
+LIBS:Altera
+LIBS:ESD_Protection
+LIBS:Lattice
+LIBS:Oscillators
+LIBS:Power_Management
+LIBS:Worldsemi
+LIBS:Xicor
+LIBS:Zilog
+LIBS:ac-dc
+LIBS:actel
+LIBS:adc-dac
+LIBS:analog_devices
+LIBS:analog_switches
+LIBS:atmel
+LIBS:audio
+LIBS:brooktre
+LIBS:cmos4000
+LIBS:cmos_ieee
+LIBS:conn
+LIBS:contrib
+LIBS:cypress
+LIBS:dc-dc
+LIBS:device
+LIBS:digital-audio
+LIBS:diode
+LIBS:display
+LIBS:dsp
+LIBS:elec-unifil
+LIBS:ftdi
+LIBS:gennum
+LIBS:graphic
+LIBS:hc11
+LIBS:intel
+LIBS:interface
+LIBS:ir
+LIBS:linear
+LIBS:logo
+LIBS:maxim
+LIBS:memory
+LIBS:microchip
+LIBS:microchip_dspic33dsc
+LIBS:microchip_pic10mcu
+LIBS:microchip_pic12mcu
+LIBS:microchip_pic16mcu
+LIBS:microchip_pic18mcu
+LIBS:microchip_pic32mcu
+LIBS:microcontrollers
+LIBS:motor_drivers
+LIBS:motorola
+LIBS:msp430
+LIBS:nordicsemi
+LIBS:nxp_armmcu
+LIBS:onsemi
+LIBS:opto
+LIBS:philips
+LIBS:power
+LIBS:powerint
+LIBS:pspice
+LIBS:references
+LIBS:regul
+LIBS:relays
+LIBS:rfcom
+LIBS:silabs
+LIBS:siliconi
+LIBS:stm8
+LIBS:stm32
+LIBS:supertex
+LIBS:switches
+LIBS:texas
+LIBS:transf
+LIBS:transistors
+LIBS:ttl_ieee
+LIBS:valves
+LIBS:video
+LIBS:xilinx
 LIBS:ciaa-nxp-cache
 EELAYER 25 0
@@
 Fuente de alimentación con rango aproximado de entrada de 12 a 30V (CC).\nTensiones de salida: 5V, 3A y 3.3V, 1A.\nPosibilidad de alimentar la CIAA a través del puerto USB mediante la conexión con D1.
 $Comp
-L NCP1117ST33T3G U2
+L NCP1117ST33T3G-RESCUE-ciaa-nxp U3
 U 1 1 581984AA
 P 7450 3650
-F 0 "U2" H 7600 3454 40  0000 C CNN
+F 0 "U3" H 7600 3454 40  0000 C CNN
 F 1 "NCP1117ST33T3G" H 7450 3850 40  0000 C CNN
 F 2 "~" H 7450 3650 60  0000 C CNN
@@
 $EndComp
 $Comp
-L LM2596-5.0 U1
+L LM2596-5.0 U2
 U 1 1 581984B1
 P 4950 3450
-F 0 "U1" H 4950 3800 60  0000 C CNN
+F 0 "U2" H 4950 3800 60  0000 C CNN
 F 1 "LM2596-5.0" H 4950 3100 60  0000 C CNN
 F 2 "~" H 4950 3450 60  0000 C CNN
@@
 $EndComp
 $Comp
-L CAPAPOL C1
+L CAPAPOL C6
 U 1 1 581984B8
 P 3500 3500
-F 0 "C1" H 3550 3600 40  0000 L CNN
+F 0 "C6" H 3550 3600 40  0000 L CNN
 F 1 "470uF" H 3550 3400 40  0000 L CNN
 F 2 "~" H 3600 3350 30  0000 C CNN
@@
 $EndComp
 $Comp
-L CAPAPOL C2
+L CAPAPOL C7
 U 1 1 581984EC
 P 6600 3850
-F 0 "C2" H 6650 3950 40  0000 L CNN
+F 0 "C7" H 6650 3950 40  0000 L CNN
 F 1 "330uF" H 6650 3750 40  0000 L CNN
 F 2 "~" H 6700 3700 30  0000 C CNN
@@
 $EndComp
 $Comp
-L CAPAPOL C3
+L CAPAPOL C8
 U 1 1 581984FF
 P 8050 3850
-F 0 "C3" H 8100 3950 40  0000 L CNN
+F 0 "C8" H 8100 3950 40  0000 L CNN
 F 1 "10uF" H 8100 3750 40  0000 L CNN
 F 2 "~" H 8150 3700 30  0000 C CNN
@@
 $EndComp
 $Comp
-L THERMISTOR TH1
+L THERMISTOR-RESCUE-ciaa-nxp TH1
 U 1 1 5819851A
 P 3200 3250
@@
 L PWR_FLAG #FLG027
 U 1 1 581985BE
-P 5700 2650
-F 0 "#FLG027" H 5700 2745 30  0001 C CNN
-F 1 "PWR_FLAG" H 5700 2830 30  0000 C CNN
-F 2 "" H 5700 2650 60  0000 C CNN
-F 3 "" H 5700 2650 60  0000 C CNN
-	1    5700 2650
-	1    0    0    -1
-$EndComp
-Wire Wire Line
-	5700 2650 5700 2700
+P 5700 2600
+F 0 "#FLG027" H 5700 2695 30  0001 C CNN
+F 1 "PWR_FLAG" H 5700 2780 30  0000 C CNN
+F 2 "" H 5700 2600 60  0000 C CNN
+F 3 "" H 5700 2600 60  0000 C CNN
+	1    5700 2600
+	1    0    0    -1
+$EndComp
+Wire Wire Line
+	5700 2600 5700 2700
 Connection ~ 5700 2700
 Text Notes 4700 4500 0    60   ~ 0
 Reemplazo SMD del 1N5825.
 $Comp
-L TB_1X2 J2
+L TB_1X2 J5
 U 1 1 581985C7
 P 1950 3350
-F 0 "J2" H 1900 3600 60  0000 C CNN
+F 0 "J5" H 1900 3600 60  0000 C CNN
 F 1 "TB_1X2" H 2000 3100 60  0000 C CNN
 F 2 "~" H 1900 3400 60  0000 C CNN
@@
 Connection ~ 5600 3650
 $Comp
-L USB_OTG P6
+L USB_OTG-RESCUE-ciaa-nxp P2
 U 1 1 5819B2D9
 P 4300 2500
-F 0 "P6" H 4625 2375 50  0000 C CNN
+F 0 "P2" H 4625 2375 50  0000 C CNN
 F 1 "USB_OTG" H 4300 2700 50  0000 C CNN
 F 2 "" V 4250 2400 50  0000 C CNN
